File: FULL ADDER 2.0/FULL ADDER 2.0.kicad_pcb (KiCad board)
At the start: 2 copper layers, 87 parts, among them J1 Barrel_Jack, SW1 SW_SPDT, SW10 SW_SPDT, SW11 SW_SPDT, SW12 SW_SPDT, SW13 SW_SPDT, SW14 SW_SPDT, SW15 SW_SPDT, SW16 SW_SPDT, SW17 SW_Push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

Commit message: nm
Parts:
- moved D1 42.1 mm to (33.3, 124.0)
- moved D2 42.1 mm to (62.0, 124.0)
- moved D5 42.1 mm to (142.3, 123.5)
- moved D4 42.1 mm to (115.3, 123.5)
- moved D10 41.5 mm to (62.0, 80.0)
- moved D11 41.5 mm to (87.5, 80.0)
- moved D12 41.5 mm to (112.7, 81.0)
- moved D13 41.5 mm to (139.5, 81.0)
- moved D14 41.5 mm to (166.0, 81.0)
- moved D15 41.5 mm to (191.2, 81.5)
- moved D16 41.5 mm to (218.2, 81.0)
- moved D9 41.5 mm to (35.5, 80.5)
- moved D3 40.6 mm to (88.5, 124.5)
- moved D6 40.6 mm to (169.5, 124.5)
- moved D8 39.6 mm to (224.0, 125.0)
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Routing:
- net GND: track 0.00 -> 1716.9 mm
- net (no net): track 0.00 -> 452.6 mm
- net VCC: track 0.00 -> 252.3 mm
- net /B7: track 0.00 -> 204.4 mm
- net /A7: track 0.00 -> 179.2 mm
- net /B4: track 0.00 -> 178.0 mm
- net /A2: track 0.00 -> 170.1 mm
- net /S3: track 0.00 -> 145.7 mm
- net /S2: track 0.00 -> 143.6 mm
- net /B0: track 0.00 -> 135.3 mm
- net Net-(D10-A): track 0.00 -> 128.8 mm
- net Net-(D2-A): track 0.00 -> 124.8 mm
- net /B6: track 0.00 -> 124.7 mm
- net /S1: track 0.00 -> 123.1 mm
- net /A0: track 0.00 -> 121.7 mm
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Other:
- board outline added: 248.5 x 171 mm
